Commit message: updating the project

File: project_goChaseIt/drive_bot/urdf/backup_drive_bot.xacro (robot description, xacro)
@@ -9,5 +9,5 @@
   </joint>
   <joint type="continuous" name="left_wheel_hinge">
-    <origin xyz="0 0.125 0" rpy="0 0 0"/>
+    <origin xyz="-0.07 0.12 0" rpy="0 0 0"/>
     <child link="left_wheel"/>
     <parent link="chassis"/>
@@ -17,5 +17,5 @@
   </joint>
   <joint type="continuous" name="right_wheel_hinge">
-    <origin xyz="0 -0.125 0" rpy="0 0 0"/>
+    <origin xyz="-0.07 -0.12 0" rpy="0 0 0"/>
     <child link="right_wheel"/>
     <parent link="chassis"/>
@@ -51,5 +51,5 @@
     <inertial>
       <mass value="5.0"/>
-      <origin xyz="0 0 0" rpy="0 1.5707 1.5707"/>
+      <origin xyz="-0 0 0" rpy="0 1.5707 1.5707"/>
       <inertia
           ixx="0.1" ixy="0" ixz="0"
@@ -61,5 +61,5 @@
       <origin xyz="0 0 0" rpy="0 1.5707 1.5707"/>
       <geometry>
-        <cylinder radius="0.1" length="0.025"/>
+        <cylinder radius="0.1" length="0.03"/>
       </geometry>
     </collision>
@@ -67,5 +67,5 @@
       <origin xyz="0 0 0" rpy="0 1.5707 1.5707"/>
       <geometry>
-        <cylinder radius="0.1" length="0.025"/>
+        <cylinder radius="0.1" length="0.03"/>
       </geometry>
     </visual>
@@ -84,5 +84,5 @@
       <origin xyz="0 0 0" rpy="0 1.5707 1.5707"/>
       <geometry>
-        <cylinder radius="0.1" length="0.025"/>
+        <cylinder radius="0.1" length="0.03"/>
       </geometry>
     </collision>
@@ -90,5 +90,5 @@
       <origin xyz="0 0 0" rpy="0 1.5707 1.5707"/>
       <geometry>
-        <cylinder radius="0.1" length="0.025"/>
+        <cylinder radius="0.1" length="0.03"/>
       </geometry>
     </visual>
