Commit message: MOD: changed the robot.xacro file to accomodate the z offset

File: project_whereAmI/drive_bot/urdf/drive_bot.xacro (robot description, xacro)
@@ -4,5 +4,5 @@
   <link name="robot_footprint"></link>
   <joint name="robot_footprint_joint" type="fixed">
-    <origin xyz="0 0 0" rpy="0 0 0" />
+    <origin xyz="0 0 0.1" rpy="0 0 0" />
     <parent link="robot_footprint"/>
     <child link="chassis" />
